Commit message: message filter

File: urdf/mobile_robot2.xacro (robot description, xacro)
@@ -8,6 +8,6 @@
   <xacro:property name="body_width"   value="0.200" />
   <xacro:property name="body_length"  value="0.400" />
-  <xacro:property name="body_mass"  value="1.0" />
-  <xacro:property name="wheel_mass"  value="0.5" />
+  <xacro:property name="body_mass"  value="0.1" />
+  <xacro:property name="wheel_mass"  value="0.05" />
    <link name="car_body">
     <visual>
@@ -109,5 +109,5 @@
     <inertial>
       <origin xyz="0 0 ${-0.5 * wheel_radius}" rpy="0 0 0"/>
-      <mass value="0.5"/>
+      <mass value="0.05"/>
       <inertia ixx="6.0e-4" ixy="0" ixz="0" iyy="6.0e-4" iyz="0" izz="6.0e-4"/>
     </inertial>
@@ -136,11 +136,11 @@
   <gazebo reference="car_body">
    <material>Gazebo/Blue</material>
-   <mu1>0.0001</mu1>
-   <mu2>0.0001</mu2>
+   <mu1>0.001</mu1>
+   <mu2>0.001</mu2>
  </gazebo>
  <gazebo reference="wheelR">
    <material>Gazebo/Green</material>
-   <mu1>100000.0</mu1>
-   <mu2>100.0</mu2>
+   <mu1>100.0</mu1>
+   <mu2>10.0</mu2>
    <kp>100000.0</kp>
    <kd>1.0</kd>
@@ -149,6 +149,6 @@
  <gazebo reference="wheelL">
    <material>Gazebo/Red</material>
-   <mu1>100000.0</mu1>
-   <mu2>100.0</mu2>
+   <mu1>100.0</mu1>
+   <mu2>10.0</mu2>
    <kp>100000.0</kp>
    <kd>1.0</kd>
@@ -157,11 +157,11 @@
   <gazebo reference="support">
    <material>Gazebo/Blue</material>
-   <mu1>0.0001</mu1>
-   <mu2>0.0001</mu2>
+   <mu1>0.001</mu1>
+   <mu2>0.001</mu2>
   </gazebo>
   <gazebo>
     <plugin name="differential_drive_controller" filename="libgazebo_ros_diff_drive.so">
       <alwaysOn>true</alwaysOn>
-      <updateRate>10</updateRate>
+      <updateRate>100</updateRate>
       <leftJoint>jointL</leftJoint>
       <rightJoint>jointR</rightJoint>
@@ -176,10 +176,10 @@
     <plugin name="p3d_base_controller" filename="libgazebo_ros_p3d.so">
       <alwaysOn>true</alwaysOn>
-      <updateRate>10.0</updateRate>
+      <updateRate>100.0</updateRate>
       <bodyName>car_body</bodyName>
       <topicName>ground_truth/state</topicName>
-      <gaussianNoise>0.01</gaussianNoise>
+      <!--gaussianNoise>0.001</gaussianNoise -->
       <frameName>world</frameName>
-      <xyzOffsets>0 0 0</xyzOffsets>
+      <xyzOffsets>${-body_length * 0.35} 0 0</xyzOffsets>
       <rpyOffsets>0 0 0</rpyOffsets>
     </plugin>
